File: Schematic/LoRaXcvr_R2.kicad_pcb (KiCad board)
At the start: 4 copper layers, 76.2 x 63.5 mm, 57 parts, among them J1 Screw_Terminal_01x04, J10 Conn_01x08, J2 Conn_02x03_Odd_Even, J3 Conn_01x04, J4 Conn_01x02, J5 Conn_01x03, J6 Conn_01x08, J7 Conn_01x10, J8 Conn_01x06, Q1 Q_PMOS_GSD, SW1 SW_Push, U1 LP38693MP-5.0, U2 AP2125K-3.3, U3 AP2125K-3.3, U4 STM32L152CCTx, U5 RFM95W-915S2, U6 MCP131X-2X, Y1 8Mhz, Y2 32.768KHz

Commit message: Updated R2 schematic and documents
Parts:
- removed R10, R11: 0, Resistor_SMD:R_0805_2012Metric
- J1: value Screw_Terminal_01x04 -> Screw_Terminal_01x02; footprint TerminalBlock_TE-Connectivity:TerminalBlock_TE_282834-4_1x04_P2.54mm_Horizontal -> TerminalBlock_TE-Connectivity:TerminalBlock_TE_282834-2_1x02_P2.54mm_Horizontal
- moved J1 0.09 mm to (109.4, 66.2)
Connections:
- J1 pad 2: /BATV6 -> GND
Routing:
- net Net-(J2-Pad3): track 15.5 -> 5.91 mm, vias 1 -> 0
- net Net-(J2-Pad4): track 15.2 -> 7.15 mm, vias 1 -> 0
- net /BATV6: track 40.2 -> 32.6 mm
- net GND: track 67.7 -> 68.6 mm, vias 31 -> 29
Other:
- board text added: "REV"
- board text removed: "Main Board"
- board text removed: "PNWAS"
- board text removed: "REV A"
